File: keyboard-pcb-tutorial.kicad_pcb (KiCad board)
At the start: 2 copper layers, 79.4 x 38.1 mm, 24 parts, among them SW1 SW_Push, U1 ATmega32U4-A, Y1 16MHz

Commit message: Added routing
Connections:
- U1 pad 27: unconnected-(U1-Pad27) -> ROW0
- U1 pad 28: unconnected-(U1-Pad28) -> COL1
- U1 pad 29: unconnected-(U1-Pad29) -> COL0
- U1 pad 30: unconnected-(U1-Pad30) -> ROW1
Routing:
- net GND: track 0.00 -> 139.7 mm
- net +5V: track 0.00 -> 98.0 mm, vias 0 -> 5
- net COL1: track 0.00 -> 54.5 mm
- net ROW1: track 0.00 -> 50.0 mm
- net ROW0: track 0.00 -> 48.1 mm
- net Net-(R3-Pad2): track 0.00 -> 40.9 mm, vias 0 -> 3
- net COL0: track 0.00 -> 35.1 mm
- net Net-(R1-Pad2): track 0.00 -> 23.3 mm
- net Net-(R2-Pad2): track 0.00 -> 22.1 mm
- net VCC: track 0.00 -> 14.9 mm
- net Net-(C2-Pad2): track 0.00 -> 11.8 mm, vias 0 -> 2
- net Net-(C3-Pad2): track 0.00 -> 8.26 mm
- net Net-(D3-Pad2): track 0.00 -> 7.14 mm
- net Net-(D1-Pad2): track 0.00 -> 6.97 mm
- net Net-(D4-Pad2): track 0.00 -> 6.82 mm
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
Commit message: Finish the design
Routing:
- added copper zone on B.Cu, net GND
Other:
- board text added: "TecktTest v1.0"
Changed lines of the file:
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@@
   (gr_arc (start 59.53125 89.69375) (mid 60.228702 88.009952) (end 61.9125 87.3125) (layer "Edge.Cuts") (width 0.1))
   (gr_line (start 138.90625 89.69375) (end 138.90625 123.03125) (layer "Edge.Cuts") (width 0.1))
+  (gr_text "TecktTest v1.0" (at 93.6625 123.03125) (layer "B.SilkS")
+    (effects (font (size 1 1) (thickness 0.15)) (justify mirror))
+  )
   (segment (start 88.9 118.26875) (end 94.45625 112.7125) (width 0.381) (layer "F.Cu") (net 1))
   (segment (start 83.3225 108.74375) (end 83.34375 108.7225) (width 0.381) (layer "F.Cu") (net 1))
@@
   (segment (start 96.8375 110.2125) (end 96.6875 110.3625) (width 0.254) (layer "B.Cu") (net 20))
   (segment (start 96.6875 110.3625) (end 93.0125 110.3625) (width 0.254) (layer "B.Cu") (net 20))
+  (zone (net 2) (net_name "GND") (layer "B.Cu") (hatch edge 0.508)
+    (connect_pads (clearance 0.508))
+    (min_thickness 0.254) (filled_areas_thickness no)
+    (fill yes (thermal_gap 0.508) (thermal_bridge_width 0.508))
+    (polygon
+      (pts
+        (xy 138.90625 125.4125)
+        (xy 59.53125 125.4125)
+        (xy 59.53125 87.3125)
+        (xy 138.90625 87.3125)
+      )
+    )
+  )
 )
